File: fabrication/plates/corne-eclipse-universal-plates-mx-or-chocv2-1.5mm.kicad_pcb (KiCad board)
At the start: 2 copper layers, 272.4 x 180.5 mm, 4 parts

Commit message: feat(fabrication): add universal, choc v1/v2, and mx board variants
- Custom universal switch footprint (MX + Choc v1/v2 hotswap, south-facing)
- Separate Choc v1/v2 footprint (compact pads, no MX overlap)
- Separate MX-only footprint
- Three PCB variants: universal, choc, mx
- Choc and MX plate variants with mouse bite bridges
- Custom tenting puck (no center hole, smaller annular rings)
- EC11 encoder swapped to EC12E
- LED pad remapping for marbastlib Choc LED footprint
- Silkscreen cleanup on MCU, encoders, reset, JST, nice!view
- All net assignments verified against original

Co-Authored-By: Claude Opus 4.6 (1M context) <noreply@anthropic.com>
Parts:
- added REF**: BreakLine_2h_D0.5mm_P0.85mm, Panelization:BreakLine_2h_D0.5mm_P0.85mm, F.Cu at (160.1, 82.2)
- added REF**: BreakLine_2h_D0.5mm_P0.85mm, Panelization:BreakLine_2h_D0.5mm_P0.85mm, F.Cu at (209.4, 107.7)
- added REF**: BreakLine_2h_D0.5mm_P0.85mm, Panelization:BreakLine_2h_D0.5mm_P0.85mm, F.Cu at (124.3, 52.9)
- added REF**: BreakLine_2h_D0.5mm_P0.85mm, Panelization:BreakLine_2h_D0.5mm_P0.85mm, F.Cu at (147.3, 51.1)
- added REF**: BreakLine_2h_D0.5mm_P0.85mm, Panelization:BreakLine_2h_D0.5mm_P0.85mm, F.Cu at (61.1, 96.8)
- added REF**: BreakLine_2h_D0.5mm_P0.85mm, Panelization:BreakLine_2h_D0.5mm_P0.85mm, F.Cu at (160.1, 114.7)
- added REF**: BreakLine_2h_D0.5mm_P0.85mm, Panelization:BreakLine_2h_D0.5mm_P0.85mm, F.Cu at (61.1, 109.9)
- added REF**: BreakLine_2h_D0.5mm_P0.85mm, Panelization:BreakLine_2h_D0.5mm_P0.85mm, F.Cu at (147.5, 142.5)
- added REF**: BreakLine_2h_D0.5mm_P0.85mm, Panelization:BreakLine_2h_D0.5mm_P0.85mm, F.Cu at (161.8, 82.2)
- added REF**: BreakLine_2h_D0.5mm_P0.85mm, Panelization:BreakLine_2h_D0.5mm_P0.85mm, F.Cu at (124.4, 142.5)
- added REF**: BreakLine_2h_D0.5mm_P0.85mm, Panelization:BreakLine_2h_D0.5mm_P0.85mm, F.Cu at (124.3, 51.2)
- added REF**: BreakLine_2h_D0.5mm_P0.85mm, Panelization:BreakLine_2h_D0.5mm_P0.85mm, F.Cu at (149.5, 51.1)
- added REF**: BreakLine_2h_D0.5mm_P0.85mm, Panelization:BreakLine_2h_D0.5mm_P0.85mm, F.Cu at (127.4, 52.9)
- added REF**: BreakLine_2h_D0.5mm_P0.85mm, Panelization:BreakLine_2h_D0.5mm_P0.85mm, F.Cu at (158.3, 82.2)
- added REF**: BreakLine_2h_D0.5mm_P0.85mm, Panelization:BreakLine_2h_D0.5mm_P0.85mm, F.Cu at (161.8, 114.7)
- added REF**: BreakLine_2h_D0.5mm_P0.85mm, Panelization:BreakLine_2h_D0.5mm_P0.85mm, F.Cu at (127.5, 139.0)
- added REF**: BreakLine_2h_D0.5mm_P0.85mm, Panelization:BreakLine_2h_D0.5mm_P0.85mm, F.Cu at (147.3, 52.8)
- added REF**: BreakLine_2h_D0.5mm_P0.85mm, Panelization:BreakLine_2h_D0.5mm_P0.85mm, F.Cu at (211.1, 96.8)
- added REF**: BreakLine_2h_D0.5mm_P0.85mm, Panelization:BreakLine_2h_D0.5mm_P0.85mm, F.Cu at (149.6, 140.8)
- added REF**: BreakLine_2h_D0.5mm_P0.85mm, Panelization:BreakLine_2h_D0.5mm_P0.85mm, F.Cu at (124.4, 140.7)
- added REF**: BreakLine_2h_D0.5mm_P0.85mm, Panelization:BreakLine_2h_D0.5mm_P0.85mm, F.Cu at (147.5, 139.0)
- added REF**: BreakLine_2h_D0.5mm_P0.85mm, Panelization:BreakLine_2h_D0.5mm_P0.85mm, F.Cu at (62.9, 96.8)
- added REF**: BreakLine_2h_D0.5mm_P0.85mm, Panelization:BreakLine_2h_D0.5mm_P0.85mm, F.Cu at (64.6, 109.9)
- added REF**: BreakLine_2h_D0.5mm_P0.85mm, Panelization:BreakLine_2h_D0.5mm_P0.85mm, F.Cu at (127.5, 142.5)
- added REF**: BreakLine_2h_D0.5mm_P0.85mm, Panelization:BreakLine_2h_D0.5mm_P0.85mm, F.Cu at (124.3, 49.4)
- added REF**: BreakLine_2h_D0.5mm_P0.85mm, Panelization:BreakLine_2h_D0.5mm_P0.85mm, F.Cu at (209.3, 96.8)
- added REF**: BreakLine_2h_D0.5mm_P0.85mm, Panelization:BreakLine_2h_D0.5mm_P0.85mm, F.Cu at (147.3, 49.3)
- added REF**: BreakLine_2h_D0.5mm_P0.85mm, Panelization:BreakLine_2h_D0.5mm_P0.85mm, F.Cu at (149.5, 52.9)
- added REF**: BreakLine_2h_D0.5mm_P0.85mm, Panelization:BreakLine_2h_D0.5mm_P0.85mm, F.Cu at (147.5, 140.8)
- added REF**: BreakLine_2h_D0.5mm_P0.85mm, Panelization:BreakLine_2h_D0.5mm_P0.85mm, F.Cu at (127.5, 140.8)
- added REF**: BreakLine_2h_D0.5mm_P0.85mm, Panelization:BreakLine_2h_D0.5mm_P0.85mm, F.Cu at (149.6, 142.5)
- added REF**: BreakLine_2h_D0.5mm_P0.85mm, Panelization:BreakLine_2h_D0.5mm_P0.85mm, F.Cu at (212.9, 107.7)
- added REF**: BreakLine_2h_D0.5mm_P0.85mm, Panelization:BreakLine_2h_D0.5mm_P0.85mm, F.Cu at (149.6, 139.0)
- added REF**: BreakLine_2h_D0.5mm_P0.85mm, Panelization:BreakLine_2h_D0.5mm_P0.85mm, F.Cu at (158.3, 114.7)
- added REF**: BreakLine_2h_D0.5mm_P0.85mm, Panelization:BreakLine_2h_D0.5mm_P0.85mm, F.Cu at (127.4, 49.4)
- added REF**: BreakLine_2h_D0.5mm_P0.85mm, Panelization:BreakLine_2h_D0.5mm_P0.85mm, F.Cu at (124.4, 139.0)
- added REF**: BreakLine_2h_D0.5mm_P0.85mm, Panelization:BreakLine_2h_D0.5mm_P0.85mm, F.Cu at (211.1, 107.7)
- added REF**: BreakLine_2h_D0.5mm_P0.85mm, Panelization:BreakLine_2h_D0.5mm_P0.85mm, F.Cu at (64.6, 96.8)
- added REF**: BreakLine_2h_D0.5mm_P0.85mm, Panelization:BreakLine_2h_D0.5mm_P0.85mm, F.Cu at (127.4, 51.1)
- added REF**: BreakLine_2h_D0.5mm_P0.85mm, Panelization:BreakLine_2h_D0.5mm_P0.85mm, F.Cu at (62.8, 109.9)
- added REF**: BreakLine_2h_D0.5mm_P0.85mm, Panelization:BreakLine_2h_D0.5mm_P0.85mm, F.Cu at (212.8, 96.8)
- added REF**: BreakLine_2h_D0.5mm_P0.85mm, Panelization:BreakLine_2h_D0.5mm_P0.85mm, F.Cu at (149.5, 49.4)
- moved REF** 6.93 mm to (276.5, 174.6)
- moved REF** 6.93 mm to (276.3, 85.6)
Other:
- outline, holes or cut-outs redrawn
