File: fabrication/circuitboard/corne-eclipse-mx.kicad_pcb (KiCad board)
At the start: 2 copper layers, 275.5 x 105.6 mm, 182 parts, among them J2 OLED, J4 OLED, SW1 SW_MX_HS, SW10 SW_MX_HS, SW11 SW_MX_HS, SW12 SW_MX_HS, SW13 SW_MX_HS, SW14 SW_MX_HS, SW15 SW_MX_HS, SW16 SW_MX_HS, SW17 SW_MX_HS, SW18 SW_MX_HS, SW2 SW_MX_HS, SW20 SW_MX_HS, SW21 SW_MX_HS, SW22 SW_MX_HS, SW23 SW_MX_HS, SW24 SW_MX_HS, SW25 SW_MX_HS, SW26 SW_MX_HS, SW27 SW_MX_HS, SW28 SW_MX_HS, SW29 SW_MX_HS, SW3 SW_MX_HS, SW30 SW_MX_HS, SW31 SW_MX_HS, SW32 SW_MX_HS, SW33 SW_MX_HS, SW34 SW_MX_HS, SW35 SW_MX_HS, SW36 SW_MX_HS, SW37 SW_MX_HS, SW38 SW_MX_HS, SW39 SW_MX_HS, SW4 SW_MX_HS, SW40 SW_MX_HS, SW42 SW_MX_HS, SW43 SW_MX_HS, SW44 SW_MX_HS, SW5 SW_MX_HS, SW6 SW_MX_HS, SW7 SW_MX_HS, SW8 SW_MX_HS, SW9 SW_MX_HS, U1 nice!nano, U2 nice!nano

Commit message: wip:pcbs
Parts:
- moved D19B 21.6 mm to (57.4, 85.0)
- moved D40B 21.2 mm to (239.4, 85.3)
- moved D21 0.59 mm to (136.3, 91.9), turned to 150 degrees
- moved D41 0.50 mm to (160.6, 91.8)
Changed lines of the file:
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@@
 	(footprint "kbd:D3_SMD_v2"
 		(layer "B.Cu")
-		(at 135.8575 91.53 -30)
+		(at 136.320305 91.8925 150)
 		(descr "Resitance 3 pas")
 		(tags "R")
 		(property "Reference" "D21"
-			(at 0.5 0 150)
+			(at 0.500001 -0.000001 150)
 			(layer "B.Fab")
 			(hide yes)
@@
 		(duplicate_pad_numbers_are_jumpers no)
 		(fp_line
-			(start -2.7 0.75)
-			(end -2.7 -0.75)
+			(start 2.7 0.75)
+			(end 2.7 -0.75)
 			(stroke
 				(width 0.15)
@@
 		)
 		(fp_line
-			(start -2.7 -0.75)
-			(end 2.7 -0.75)
+			(start 2.7 0.75)
+			(end -2.7 0.75)
 			(stroke
 				(width 0.15)
@@
 		)
 		(fp_line
-			(start -0.5 0.5)
-			(end -0.5 -0.5)
+			(start 0.499999 -0.5)
+			(end -0.4 0)
 			(stroke
 				(width 0.15)
@@
 		)
 		(fp_line
-			(start -0.4 0)
-			(end 0.5 0.5)
+			(start 0.5 0.499999)
+			(end 0.499999 -0.5)
 			(stroke
 				(width 0.15)
@@
 		)
 		(fp_line
-			(start 0.5 0.5)
-			(end 0.5 -0.5)
+			(start -0.4 0)
+			(end 0.5 0.499999)
 			(stroke
 				(width 0.15)
@@
 		)
 		(fp_line
-			(start 0.5 -0.5)
-			(end -0.4 0)
+			(start -0.499999 0.5)
+			(end -0.5 -0.499999)
 			(stroke
 				(width 0.15)
@@
 		)
 		(fp_line
-			(start 2.7 0.75)
-			(end -2.7 0.75)
+			(start -2.7 -0.75)
+			(end 2.7 -0.75)
 			(stroke
 				(width 0.15)
@@
 		)
 		(fp_line
-			(start 2.7 0.75)
-			(end 2.7 -0.75)
+			(start -2.7 0.75)
+			(end -2.7 -0.75)
 			(stroke
 				(width 0.15)
@@
 		)
 		(pad "1" smd rect
-			(at -1.775 0 330)
+			(at -1.775 0 150)
 			(size 1.4 1)
 			(layers "B.Cu" "B.Mask" "B.Paste")
@@
 		)
 		(pad "2" smd rect
-			(at 1.775 0 330)
+			(at 1.775 0 150)
 			(size 1.4 1)
 			(layers "B.Cu" "B.Mask" "B.Paste")
@@
 	(footprint "kbd:D3_SMD_v2"
 		(layer "B.Cu")
-		(at 161.1075 91.78 30)
+		(at 160.6075 91.78 30)
 		(descr "Resitance 3 pas")
 		(tags "R")
@@
 		(tags "SOT-23 MOSFET P-Channel")
 		(property "Reference" "RGBMOS"
-			(at 0 -2.5 90)
+			(at 0 -2.5 0)
 			(layer "B.SilkS")
 			(hide yes)
@@
 		)
 		(property "Value" "AO3401A"
-			(at 0 2.5 90)
+			(at 0 2.5 0)
 			(layer "B.Fab")
 			(hide yes)
@@
 		)
 		(property "Datasheet" ""
-			(at 0 0 90)
+			(at 0 0 0)
 			(layer "B.Fab")
 			(hide yes)
@@
 		)
 		(property "Description" "AO3401A P-Ch MOSFET 30V 4A SOT-23-3 - LED power switch"
-			(at 0 0 90)
+			(at 0 0 0)
 			(layer "B.Fab")
 			(hide yes)
@@
 		)
 		(fp_text user "RGB"
-			(at 3.55 0 90)
+			(at 3.55 0 0)
 			(layer "B.SilkS")
 			(effects
@@
 		)
 		(fp_text user "MOS"
-			(at 2.55 0 90)
+			(at 2.55 0 0)
 			(layer "B.SilkS")
 			(effects
@@
 	(footprint "kbd:D3_SMD_v2"
 		(layer "B.Cu")
-		(at 218.6075 89.53 90)
+		(at 239.3575 85.28 90)
 		(descr "Resitance 3 pas")
 		(tags "R")
@@
 		(tags "SOT-23 MOSFET P-Channel")
 		(property "Reference" "RGBMOS"
-			(at 0 -2.5 90)
+			(at 0 -2.5 0)
 			(layer "B.SilkS")
 			(hide yes)
@@
 		)
 		(property "Value" "AO3401A"
-			(at 0 2.5 90)
+			(at 0 2.5 0)
 			(layer "B.Fab")
 			(hide yes)
@@
 		)
 		(property "Datasheet" ""
-			(at 0 0 90)
+			(at 0 0 0)
 			(layer "B.Fab")
 			(hide yes)
@@
 		)
 		(property "Description" "AO3401A P-Ch MOSFET 30V 4A SOT-23-3 - LED power switch"
-			(at 0 0 90)
+			(at 0 0 0)
 			(layer "B.Fab")
 			(hide yes)
@@
 		)
 		(fp_text user "RGB"
-			(at 3.55 0 90)
+			(at 3.55 0 0)
 			(layer "B.SilkS")
 			(effects
@@
 		)
 		(fp_text user "MOS"
-			(at 2.55 0 90)
+			(at 2.55 0 0)
 			(layer "B.SilkS")
 			(effects
@@
 	(footprint "kbd:D3_SMD_v2"
 		(layer "B.Cu")
-		(at 78.3575 90.005 90)
+		(at 57.3575 85.03 90)
 		(descr "Resitance 3 pas")
 		(tags "R")

Commit message: wip: pcbs
Other:
- board text added: "Design by Frosthaven Inspired by foostan's crkbd MX South Hotswap"
- board text removed: "Design by Frosthaven Inspired by foostan's crkbd MX Hotswap"
Changed lines of the file:
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@@
 		(layer "User.3")
 	)
-	(gr_text "Design by Frosthaven\nInspired by foostan's crkbd\nMX Hotswap"
-		(at 119.3575 84.53 0)
+	(gr_text "Design by Frosthaven\nInspired by foostan's crkbd\nMX South Hotswap"
+		(at 121.3575 84.53 0)
 		(layer "B.SilkS")
 		(effects
@@
 		)
 	)
-	(gr_text "Design by Frosthaven\nInspired by foostan's crkbd\nMX Hotswap"
-		(at 177.3625 84.53 0)
+	(gr_text "Design by Frosthaven\nInspired by foostan's crkbd\nMX South Hotswap"
+		(at 175.3625 84.53 0)
 		(layer "B.SilkS")
 		(effects
