File: fabrication/circuitboard/corne-eclipse-choc.kicad_pcb (KiCad board)
At the start: 2 copper layers, 275.5 x 105.6 mm, 182 parts, among them J2 OLED, J4 OLED, SW1 SW_Choc_v1v2_HS, SW10 SW_Choc_v1v2_HS, SW11 SW_Choc_v1v2_HS, SW12 SW_Choc_v1v2_HS, SW13 SW_Choc_v1v2_HS, SW14 SW_Choc_v1v2_HS, SW15 SW_Choc_v1v2_HS, SW16 SW_Choc_v1v2_HS, SW17 SW_Choc_v1v2_HS, SW18 SW_Choc_v1v2_HS, SW2 SW_Choc_v1v2_HS, SW20 SW_Choc_v1v2_HS, SW21 SW_Choc_v1v2_HS, SW22 SW_Choc_v1v2_HS, SW23 SW_Choc_v1v2_HS, SW24 SW_Choc_v1v2_HS, SW25 SW_Choc_v1v2_HS, SW26 SW_Choc_v1v2_HS, SW27 SW_Choc_v1v2_HS, SW28 SW_Choc_v1v2_HS, SW29 SW_Choc_v1v2_HS, SW3 SW_Choc_v1v2_HS, SW30 SW_Choc_v1v2_HS, SW31 SW_Choc_v1v2_HS, SW32 SW_Choc_v1v2_HS, SW33 SW_Choc_v1v2_HS, SW34 SW_Choc_v1v2_HS, SW35 SW_Choc_v1v2_HS, SW36 SW_Choc_v1v2_HS, SW37 SW_Choc_v1v2_HS, SW38 SW_Choc_v1v2_HS, SW39 SW_Choc_v1v2_HS, SW4 SW_Choc_v1v2_HS, SW40 SW_Choc_v1v2_HS, SW42 SW_Choc_v1v2_HS, SW43 SW_Choc_v1v2_HS, SW44 SW_Choc_v1v2_HS, SW5 SW_Choc_v1v2_HS, SW6 SW_Choc_v1v2_HS, SW7 SW_Choc_v1v2_HS, SW8 SW_Choc_v1v2_HS, SW9 SW_Choc_v1v2_HS, U1 nice!nano, U2 nice!nano

Commit message: wip:pcbs
Parts:
- moved D40B 5.32 mm to (239.1, 85.3)
- moved D19B 2.02 mm to (57.1, 85.5)
Changed lines of the file:
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@@
 	(footprint "kbd:D3_SMD_v2"
 		(layer "B.Cu")
-		(at 236.6075 80.555 90)
+		(at 239.1075 85.255 90)
 		(descr "Resitance 3 pas")
 		(tags "R")
@@
 	(footprint "kbd:D3_SMD_v2"
 		(layer "B.Cu")
-		(at 56.8575 87.505 90)
+		(at 57.1075 85.505 90)
 		(descr "Resitance 3 pas")
 		(tags "R")

Commit message: wip(pcbs): set board thicknesses
Other:
- copper layers 2 -> 4
Changed lines of the file:
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@@
 	(layers
 		(0 "F.Cu" signal)
-		(2 "B.Cu" signal)
+		(1 "In1.Cu" signal)
+		(2 "In2.Cu" signal)
+		(31 "B.Cu" signal)
 		(9 "F.Adhes" user "F.Adhesive")
 		(11 "B.Adhes" user "B.Adhesive")
@@
 	)
 	(setup
+		(stackup
+			(layer "F.Cu"
+				(type "copper")
+				(thickness 0.035)
+			)
+			(layer "dielectric 1"
+				(type "prepreg")
+				(thickness 0.1)
+				(material "FR4")
+				(epsilon_r 4.5)
+				(loss_tangent 0.02)
+			)
+			(layer "In1.Cu"
+				(type "copper")
+				(thickness 0.0175)
+			)
+			(layer "dielectric 2"
+				(type "core")
+				(thickness 1.265)
+				(material "FR4")
+				(epsilon_r 4.5)
+				(loss_tangent 0.02)
+			)
+			(layer "In2.Cu"
+				(type "copper")
+				(thickness 0.0175)
+			)
+			(layer "dielectric 3"
+				(type "prepreg")
+				(thickness 0.1)
+				(material "FR4")
+				(epsilon_r 4.5)
+				(loss_tangent 0.02)
+			)
+			(layer "B.Cu"
+				(type "copper")
+				(thickness 0.035)
+			)
+			(copper_finish "ENIG")
+			(dielectric_constraints no)
+			(board_thickness 1.6)
+		)
 		(pad_to_mask_clearance 0)
 		(allow_soldermask_bridges_in_footprints no)

Commit message: wip(pcbs): added pour layers for power/ground
Routing:
- added copper zone on In1.Cu, net GND
- added copper zone on In1.Cu, net GNDA
- added copper zone on In2.Cu, net LED_PWR
- added copper zone on In2.Cu, net LED_PWR_r
Other:
- outline, holes or cut-outs redrawn
