File: fabrication/circuitboard/corne-eclipse-mx-south.kicad_pcb (KiCad board)
At the start: 4 copper layers, 275.5 x 105.6 mm, 182 parts, among them J2 OLED, J4 OLED, SW1 SW_MX_HS, SW10 SW_MX_HS, SW11 SW_MX_HS, SW12 SW_MX_HS, SW13 SW_MX_HS, SW14 SW_MX_HS, SW15 SW_MX_HS, SW16 SW_MX_HS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

Commit message: wip(pcbs): added pour layers for power/ground
Routing:
- added copper zone on In1.Cu, net GND
- added copper zone on In1.Cu, net GNDA
- added copper zone on In2.Cu, net LED_PWR
- added copper zone on In2.Cu, net LED_PWR_r
Other:
- outline, holes or cut-outs redrawn
