File: fabrication/circuitboard/corne-eclipse-mx-north.kicad_pcb (KiCad board)
At the start: 2 copper layers, 275.5 x 105.6 mm, 182 parts, among them J2 OLED, J4 OLED, SW1 SW_MX_HS, SW10 SW_MX_HS, SW11 SW_MX_HS, SW12 SW_MX_HS, SW13 SW_MX_HS, SW14 SW_MX_HS, SW15 SW_MX_HS, SW16 SW_MX_HS, SW17 SW_MX_HS, SW18 SW_MX_HS, SW2 SW_MX_HS, SW20 SW_MX_HS, SW21 SW_MX_HS, SW22 SW_MX_HS, SW23 SW_MX_HS, SW24 SW_MX_HS, SW25 SW_MX_HS, SW26 SW_MX_HS, SW27 SW_MX_HS, SW28 SW_MX_HS, SW29 SW_MX_HS, SW3 SW_MX_HS, SW30 SW_MX_HS, SW31 SW_MX_HS, SW32 SW_MX_HS, SW33 SW_MX_HS, SW34 SW_MX_HS, SW35 SW_MX_HS, SW36 SW_MX_HS, SW37 SW_MX_HS, SW38 SW_MX_HS, SW39 SW_MX_HS, SW4 SW_MX_HS, SW40 SW_MX_HS, SW42 SW_MX_HS, SW43 SW_MX_HS, SW44 SW_MX_HS, SW5 SW_MX_HS, SW6 SW_MX_HS, SW7 SW_MX_HS, SW8 SW_MX_HS, SW9 SW_MX_HS, U1 nice!nano, U2 nice!nano

Commit message: feat(pcb): split mx design into north-facing and south-facing
Parts:
- moved D16 17.0 mm to (68.1, 69.3)
- moved D15 17.0 mm to (49.1, 71.5)
- moved D17 17.0 mm to (87.1, 71.5)
- moved D18 16.5 mm to (106.6, 74.0)
- moved D2 16.5 mm to (33.6, 44.8)
- moved D11 16.5 mm to (90.6, 59.0)
- moved D8 16.5 mm to (33.9, 64.0)
- moved D12 16.4 mm to (109.9, 61.5)
- moved D5 16.3 mm to (90.6, 39.8)
- moved D9 16.3 mm to (52.6, 58.8)
- moved D1 16.3 mm to (14.9, 44.8)
- moved D7 16.3 mm to (14.9, 63.8)
- moved D10 16.2 mm to (71.9, 56.5)
- moved D6 16.2 mm to (109.9, 42.3)
- moved D41 15.8 mm to (171.1, 103.5)
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Other:
- board text added: "Design by Frosthaven Inspired by foostan's crkbd MX North Hotswap"
- board text removed: "Design by Frosthaven Inspired by foostan's crkbd MX South Hotswap"

Commit message: wip(pcbs): set board thicknesses
Other:
- copper layers 2 -> 4
Changed lines of the file:
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@@
 	(layers
 		(0 "F.Cu" signal)
-		(2 "B.Cu" signal)
+		(1 "In1.Cu" signal)
+		(2 "In2.Cu" signal)
+		(31 "B.Cu" signal)
 		(9 "F.Adhes" user "F.Adhesive")
 		(11 "B.Adhes" user "B.Adhesive")
@@
 	)
 	(setup
+		(stackup
+			(layer "F.Cu"
+				(type "copper")
+				(thickness 0.035)
+			)
+			(layer "dielectric 1"
+				(type "prepreg")
+				(thickness 0.1)
+				(material "FR4")
+				(epsilon_r 4.5)
+				(loss_tangent 0.02)
+			)
+			(layer "In1.Cu"
+				(type "copper")
+				(thickness 0.0175)
+			)
+			(layer "dielectric 2"
+				(type "core")
+				(thickness 1.265)
+				(material "FR4")
+				(epsilon_r 4.5)
+				(loss_tangent 0.02)
+			)
+			(layer "In2.Cu"
+				(type "copper")
+				(thickness 0.0175)
+			)
+			(layer "dielectric 3"
+				(type "prepreg")
+				(thickness 0.1)
+				(material "FR4")
+				(epsilon_r 4.5)
+				(loss_tangent 0.02)
+			)
+			(layer "B.Cu"
+				(type "copper")
+				(thickness 0.035)
+			)
+			(copper_finish "ENIG")
+			(dielectric_constraints no)
+			(board_thickness 1.6)
+		)
 		(pad_to_mask_clearance 0)
 		(allow_soldermask_bridges_in_footprints no)

Commit message: wip(pcbs): added pour layers for power/ground
Routing:
- added copper zone on In1.Cu, net GND
- added copper zone on In1.Cu, net GNDA
- added copper zone on In2.Cu, net LED_PWR
- added copper zone on In2.Cu, net LED_PWR_r
Other:
- outline, holes or cut-outs redrawn

Commit message: feat(pcbs): finished ground and led power planes on all 3
Parts:
- moved GLOW06 48.5 mm to (135.1, 29.1), turned to 0 degrees
- moved GLOW06 48.3 mm to (161.8, 29.1), turned to 0 degrees
- moved GLOW05 38.9 mm to (88.0, 25.6), turned to 90 degrees
- moved GLOW05 38.7 mm to (208.9, 25.6), turned to 90 degrees
- moved GLOW03 32.1 mm to (15.3, 64.1)
- moved GLOW03 30.0 mm to (279.3, 63.7)
- moved D28 11.5 mm to (271.1, 67.8)
- moved D7 10.5 mm to (25.4, 64.1)
- moved GLOW01 0.16 mm to (178.9, 96.6), turned to 90 degrees
- moved GLOW02 0.16 mm to (231.8, 77.9)
- moved GLOW04 0.16 mm to (267.4, 32.2), turned to 90 degrees
Routing:
- net LED_PWR: track 0.00 -> 30.1 mm, vias 0 -> 28
- net LED_PWR_r: track 0.00 -> 29.9 mm, vias 0 -> 28
- net GND: track 0.00 -> 29.6 mm, vias 0 -> 28
- net GNDA: track 0.00 -> 28.6 mm, vias 0 -> 28
