File: fabrication/circuitboard/corne-eclipse-choc-reversible.kicad_pcb (KiCad board)
At the start: 4 copper layers, 150.6 x 105.7 mm, 91 parts, among them J2 OLED, SW1 SW_Choc_v1v2_HS, SW10 SW_Choc_v1v2_HS, SW11 SW_Choc_v1v2_HS, SW12 SW_Choc_v1v2_HS, SW13 SW_Choc_v1v2_HS, SW14 SW_Choc_v1v2_HS, SW15 SW_Choc_v1v2_HS, SW16 SW_Choc_v1v2_HS, SW17 SW_Choc_v1v2_HS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

Commit message: wip(pcbs): reversible footprints and choc progress
Parts:
- ENC1: footprint Corne Eclipse:ENC_SW_EC12_Choc_v1v2_HS_1u -> reversible:ENC_SW_EC12_Choc-reversible
- J2: footprint corne:nice!view -> reversible:niceview-reversible
- PWR1: footprint corne:power -> reversible:PowerSW-reversible
- RSW1: footprint kbd:ResetSW_1side -> reversible:ResetSW-reversible
- moved PWR1 3.75 mm to (139.3, 74.9)
- moved JST 1.37 mm to (133.7, 70.3)
- moved J2 0.56 mm to (129.9, 63.1)

Commit message: wip(pcbs): reversible
Parts:
- R1: footprint Resistor_SMD:R_1206_3216Metric -> reversible:R_1206-reversible
- RGBMOS: footprint Package_TO_SOT_SMD:SOT-23 -> reversible:SOT-23-reversible
- moved D18 1.57 mm to (122.9, 65.2)
- moved R1 0.69 mm to (126.9, 69.7)
- moved D17 0.61 mm to (105.7, 66.0)
- moved RGBMOS 0.35 mm to (126.9, 66.0), turned to 0 degrees
