File: fabrication/circuitboard/corne-eclipse-choc-reversible.kicad_pcb (KiCad board)
At the start: 4 copper layers, 150.6 x 105.7 mm, 91 parts, among them J2 OLED, SW1 SW_Choc_v1v2_HS, SW10 SW_Choc_v1v2_HS, SW11 SW_Choc_v1v2_HS, SW12 SW_Choc_v1v2_HS, SW13 SW_Choc_v1v2_HS, SW14 SW_Choc_v1v2_HS, SW15 SW_Choc_v1v2_HS, SW16 SW_Choc_v1v2_HS, SW17 SW_Choc_v1v2_HS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

Commit message: wip(pcbs): wiring
Parts:
- moved D19B 18.9 mm to (75.1, 78.8), turned to 180 degrees
- moved D19 1.27 mm to (78.6, 85.3)
- moved J2 0.13 mm to (129.7, 63.1)
- turned SHINE01 to 0 degrees
- turned SHINE02 to 0 degrees
- turned SHINE03 to 0 degrees
- turned SHINE04 to 0 degrees
- turned SHINE05 to 0 degrees
- turned SHINE06 to 0 degrees
- turned SHINE13 to 0 degrees
- turned SHINE14 to 0 degrees
- turned SHINE15 to 0 degrees
- turned SHINE16 to 0 degrees
- turned SHINE17 to 0 degrees
- turned SHINE18 to 0 degrees
Routing:
- net col0: track 0.00 -> 151.5 mm, vias 0 -> 1
- net col1: track 0.00 -> 125.7 mm, vias 0 -> 2
- net Net-(U1-Pad11): track 0.00 -> 120.5 mm, vias 0 -> 1
- net col4: track 0.00 -> 107.1 mm
- net col3: track 25.7 -> 118.8 mm, vias 1 -> 0
- net Net-(U1-Pad12): track 0.00 -> 92.4 mm, vias 0 -> 2
- net col2: track 47.5 -> 139.0 mm
- net col5: track 0.00 -> 65.4 mm
- net Net-(U1-Pad24): track 0.00 -> 50.1 mm
- net row3: track 85.0 -> 130.3 mm, vias 1 -> 0
- net reset: track 0.00 -> 44.0 mm
- net VCC: track 0.00 -> 43.0 mm
- net SDA: track 0.00 -> 40.1 mm, vias 0 -> 2
- net SCL: track 0.00 -> 35.0 mm
- net data: track 0.00 -> 33.7 mm
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