File: fabrication/circuitboard/corne-eclipse-choc-reversible.kicad_pcb (KiCad board)
At the start: 4 copper layers, 150.6 x 105.7 mm, 91 parts, among them J2 OLED, SW1 SW_Choc_v1v2_HS, SW10 SW_Choc_v1v2_HS, SW11 SW_Choc_v1v2_HS, SW12 SW_Choc_v1v2_HS, SW13 SW_Choc_v1v2_HS, SW14 SW_Choc_v1v2_HS, SW15 SW_Choc_v1v2_HS, SW16 SW_Choc_v1v2_HS, SW17 SW_Choc_v1v2_HS, SW18 SW_Choc_v1v2_HS, SW2 SW_Choc_v1v2_HS, SW20 SW_Choc_v1v2_HS, SW21 SW_Choc_v1v2_HS, SW22 SW_Choc_v1v2_HS, SW3 SW_Choc_v1v2_HS, SW4 SW_Choc_v1v2_HS, SW5 SW_Choc_v1v2_HS, SW6 SW_Choc_v1v2_HS, SW7 SW_Choc_v1v2_HS, SW8 SW_Choc_v1v2_HS, SW9 SW_Choc_v1v2_HS, U1 nice!nano

Commit message: wip
Parts:
- moved GLOW05 1.48 mm to (86.9, 26.8)
- moved SHINE14 0.27 mm to (96.1, 63.6), turned to 0 degrees
- moved SHINE15 0.27 mm to (77.1, 61.2), turned to 0 degrees
- moved SHINE16 0.27 mm to (58.1, 63.6), turned to 0 degrees
- moved SHINE01 0.27 mm to (115.1, 27.9), turned to 0 degrees
- moved SHINE02 0.27 mm to (96.1, 25.6), turned to 0 degrees
- moved SHINE03 0.27 mm to (77.1, 23.2), turned to 0 degrees
- moved SHINE04 0.27 mm to (58.1, 25.6), turned to 0 degrees
- moved SHINE05 0.27 mm to (39.1, 30.3), turned to 0 degrees
- moved SHINE06 0.27 mm to (20.1, 30.3), turned to 0 degrees
- moved SHINE13 0.27 mm to (115.1, 66.0), turned to 0 degrees
- moved SHINE17 0.27 mm to (39.1, 68.3), turned to 0 degrees
- moved SHINE18 0.27 mm to (20.1, 68.3), turned to 0 degrees
Routing:
- net Net-(D6-Pad2): track 0.00 -> 16.4 mm
- net row0: track 0.00 -> 1.46 mm
